File: Electromiografo.sch (EAGLE design)
At the start: 37 parts, among them IC1 ESP32-WROOM-32E-N16, IC2 MCP73831T-2DCI_OT, IC3 741G3157DBVR, IC4 LP38692MP-3.3_NOPB, IC5 MCP73831T-2DCI_OT, IC6 LMV321IDBVRG4, IC7 LMV321IDBVRG4, IC8 LMV321IDBVRG4, IC9 AD8223ARMZ, J1 1981584-1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

Commit message: Archivo esquematico
Other:
- note added: "+"
- note added: "Alimentacion y Regulacion"
- note added: "BATT"
- note added: "FILTRO PASA BAJO"
- note added: "INA"
- note added: "conector de electrodos"
- moved on the sheet: C10, C5, C6, C7, C8, C9, IC6, IC7, IC8, R10, R5, R6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
