File: Electromiografo.sch (EAGLE design)
At the start: 40 parts, among them IC10 LMV321IDBVRG4, IC2 MCP73831T-2DCI_OT, IC5 REF2033AIDDCT, IC6 LMV321IDBVRG4, IC7 LMV321IDBVRG4, IC8 LMV321IDBVRG4, J3 SJ-3523-SMT-TR

Commit message: Finalizacion de PCB
Parts:
- added LED1, LED2, LED3: HSMW-C170-U0000, SamacSys_Parts:HSMW-C170-U0000
- renumbered S1 to FLASH, S2 to RESET
Connections:
- new net N$2: LED1.K, R3.2
- new net N$3: ESP32.IO48, LED3.A
- new net N$4: ESP32.IO47, LED2.A
- net +5V: now also LED1.A; no longer R3.2
- net GND: now also LED2.K, LED3.K; no longer R13.2
- net N$1: now also ESP32.IO0; no longer ESP32.IO45
- net VSS: now also R13.2
Changed lines of the file:
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@@
 <part name="GND17" library="PulseOximeterECG_AU" library_urn="urn:adsk.eagle:library:14846661" deviceset="GND" device=""/>
 <part name="+3V12" library="supply1" library_urn="urn:adsk.eagle:library:371" deviceset="+3V3" device=""/>
+<part name="CBAT" library="SamacSys_Parts" deviceset="1769" device=""/>
+<part name="FLASH" library="SamacSys_Parts" deviceset="B3U-1000PM" device=""/>
+<part name="RESET" library="SamacSys_Parts" deviceset="B3U-1000PM" device=""/>
+<part name="S3-1" library="PCM13SMTR" deviceset="PCM13SMTR" device=""/>
+<part name="VSS6" library="supply1" library_urn="urn:adsk.eagle:library:371" deviceset="VSS" device=""/>
+<part name="LED1" library="SamacSys_Parts" deviceset="HSMW-C170-U0000" device=""/>
+<part name="LED2" library="SamacSys_Parts" deviceset="HSMW-C170-U0000" device=""/>
+<part name="LED3" library="SamacSys_Parts" deviceset="HSMW-C170-U0000" device=""/>
 <part name="GND18" library="PulseOximeterECG_AU" library_urn="urn:adsk.eagle:library:14846661" deviceset="GND" device=""/>
-<part name="CBAT" library="SamacSys_Parts" deviceset="1769" device=""/>
-<part name="S1" library="SamacSys_Parts" deviceset="B3U-1000PM" device=""/>
-<part name="S2" library="SamacSys_Parts" deviceset="B3U-1000PM" device=""/>
-<part name="S3-1" library="PCM13SMTR" deviceset="PCM13SMTR" device=""/>
+<part name="GND19" library="PulseOximeterECG_AU" library_urn="urn:adsk.eagle:library:14846661" deviceset="GND" device=""/>
 </parts>
 <sheets>
@@
 <attribute name="VALUE" x="466.598" y="87.63" size="1.778" layer="96" rot="R270"/>
 </instance>
-<instance part="GND17" gate="1" x="469.9" y="73.66" smashed="yes" grouprefs="FILTRO">
-<attribute name="VALUE" x="467.36" y="71.12" size="1.778" layer="96"/>
+<instance part="GND17" gate="1" x="462.28" y="73.66" smashed="yes" grouprefs="FILTRO">
+<attribute name="VALUE" x="459.74" y="71.12" size="1.778" layer="96"/>
 </instance>
 <instance part="+3V12" gate="G$1" x="505.46" y="101.6" smashed="yes" rot="R270" grouprefs="FILTRO">
 <attribute name="VALUE" x="502.92" y="96.52" size="1.778" layer="96"/>
-</instance>
-<instance part="GND18" gate="1" x="462.28" y="81.28" smashed="yes" grouprefs="FILTRO">
-<attribute name="VALUE" x="459.74" y="78.74" size="1.778" layer="96"/>
 </instance>
 <instance part="CBAT" gate="G$1" x="347.98" y="200.66" smashed="yes">
@@
 <attribute name="VALUE" x="364.49" y="205.74" size="1.778" layer="96" align="center-left"/>
 </instance>
-<instance part="S1" gate="G$1" x="195.58" y="162.56" smashed="yes" rot="MR270">
+<instance part="FLASH" gate="G$1" x="195.58" y="162.56" smashed="yes" rot="MR270">
 <attribute name="NAME" x="187.96" y="151.13" size="1.778" layer="95" rot="MR270" align="center-left"/>
 <attribute name="VALUE" x="190.5" y="153.67" size="1.778" layer="96" rot="MR270" align="center-left"/>
 </instance>
-<instance part="S2" gate="G$1" x="86.36" y="149.86" smashed="yes" rot="MR270">
+<instance part="RESET" gate="G$1" x="86.36" y="149.86" smashed="yes" rot="MR270">
 <attribute name="NAME" x="78.74" y="140.97" size="1.778" layer="95" rot="MR270" align="center-left"/>
 <attribute name="VALUE" x="81.28" y="140.97" size="1.778" layer="96" rot="MR270" align="center-left"/>
@@
 <attribute name="NAME" x="251.46978125" y="152.39021875" size="1.27245" layer="95" rot="R180"/>
 <attribute name="VALUE" x="251.46605" y="165.10906875" size="1.271509375" layer="96" rot="R180"/>
+</instance>
+<instance part="VSS6" gate="G$1" x="469.9" y="73.66" smashed="yes">
+<attribute name="VALUE" x="467.36" y="68.58" size="1.778" layer="96" rot="R90"/>
+</instance>
+<instance part="LED1" gate="G$1" x="297.18" y="196.85" smashed="yes" rot="R90">
+<attribute name="NAME" x="288.29" y="209.55" size="1.778" layer="95" rot="R90"/>
+<attribute name="VALUE" x="290.83" y="209.55" size="1.778" layer="96" rot="R90"/>
+</instance>
+<instance part="LED2" gate="G$1" x="88.9" y="99.06" smashed="yes" rot="R90">
+<attribute name="NAME" x="80.01" y="111.76" size="1.778" layer="95" rot="R90"/>
+<attribute name="VALUE" x="82.55" y="111.76" size="1.778" layer="96" rot="R90"/>
+</instance>
+<instance part="LED3" gate="G$1" x="106.68" y="111.76" smashed="yes">
+<attribute name="NAME" x="119.38" y="120.65" size="1.778" layer="95"/>
+<attribute name="VALUE" x="119.38" y="118.11" size="1.778" layer="96"/>
+</instance>
+<instance part="GND18" gate="1" x="88.9" y="93.98" smashed="yes">
+<attribute name="VALUE" x="86.36" y="91.44" size="1.778" layer="96"/>
+</instance>
+<instance part="GND19" gate="1" x="106.68" y="106.68" smashed="yes">
+<attribute name="VALUE" x="104.14" y="104.14" size="1.778" layer="96"/>
 </instance>
 </instances>
@@
 <wire x1="205.74" y1="180.34" x2="208.28" y2="180.34" width="0.1524" layer="91"/>
 <wire x1="208.28" y1="180.34" x2="208.28" y2="170.18" width="0.1524" layer="91"/>
-<pinref part="S1" gate="G$1" pin="COM"/>
+<pinref part="FLASH" gate="G$1" pin="COM"/>
 <wire x1="198.12" y1="162.56" x2="198.12" y2="170.18" width="0.1524" layer="91"/>
 </segment>
@@
 <wire x1="73.66" y1="167.64" x2="73.66" y2="154.94" width="0.1524" layer="91" grouprefs="SP32"/>
 <junction x="73.66" y="154.94" grouprefs="SP32"/>
-<pinref part="S2" gate="G$1" pin="NO"/>
+<pinref part="RESET" gate="G$1" pin="NO"/>
 <wire x1="86.36" y1="149.86" x2="86.36" y2="154.94" width="0.1524" layer="91"/>
 </segment>
@@
 </segment>
 <segment>
-<pinref part="R13" gate="G$1" pin="2"/>
-<pinref part="GND17" gate="1" pin="GND"/>
-<wire x1="469.9" y1="78.74" x2="469.9" y2="76.2" width="0.1524" layer="91" grouprefs="FILTRO"/>
-</segment>
-<segment>
 <pinref part="IC10" gate="G$1" pin="GND"/>
 <wire x1="469.9" y1="101.6" x2="467.36" y2="101.6" width="0.1524" layer="91" grouprefs="FILTRO"/>
 <wire x1="467.36" y1="101.6" x2="467.36" y2="93.98" width="0.1524" layer="91" grouprefs="FILTRO"/>
 <wire x1="467.36" y1="93.98" x2="462.28" y2="93.98" width="0.1524" layer="91" grouprefs="FILTRO"/>
+<wire x1="462.28" y1="93.98" x2="462.28" y2="76.2" width="0.1524" layer="91" grouprefs="FILTRO"/>
+<pinref part="GND17" gate="1" pin="GND"/>
+</segment>
+<segment>
+<pinref part="GND19" gate="1" pin="GND"/>
+<pinref part="LED3" gate="G$1" pin="K"/>
+<wire x1="106.68" y1="109.22" x2="106.68" y2="111.76" width="0.1524" layer="91"/>
+</segment>
+<segment>
 <pinref part="GND18" gate="1" pin="GND"/>
-<wire x1="462.28" y1="93.98" x2="462.28" y2="83.82" width="0.1524" layer="91" grouprefs="FILTRO"/>
+<pinref part="LED2" gate="G$1" pin="K"/>
+<wire x1="88.9" y1="96.52" x2="88.9" y2="99.06" width="0.1524" layer="91"/>
 </segment>
 </net>
@@
 <segment>
 <pinref part="R1" gate="G$1" pin="1"/>
-<wire x1="160.02" y1="172.72" x2="195.58" y2="172.72" width="0.1524" layer="91" grouprefs="SP32"/>
-<wire x1="195.58" y1="172.72" x2="195.58" y2="180.34" width="0.1524" layer="91" grouprefs="SP32"/>
 <wire x1="195.58" y1="180.34" x2="195.58" y2="185.42" width="0.1524" layer="91" grouprefs="SP32"/>
 <pinref part="C11" gate="G$1" pin="1"/>
 <wire x1="198.12" y1="180.34" x2="195.58" y2="180.34" width="0.1524" layer="91"/>
 <junction x="195.58" y="180.34"/>
-<pinref part="ESP32" gate="G$1" pin="IO45"/>
-<pinref part="S1" gate="G$1" pin="NO"/>
-<wire x1="195.58" y1="162.56" x2="195.58" y2="172.72" width="0.1524" layer="91"/>
-<junction x="195.58" y="172.72"/>
+<pinref part="FLASH" gate="G$1" pin="NO"/>
+<wire x1="195.58" y1="162.56" x2="195.58" y2="170.18" width="0.1524" layer="91"/>
+<pinref part="ESP32" gate="G$1" pin="IO0"/>
+<wire x1="195.58" y1="170.18" x2="195.58" y2="180.34" width="0.1524" layer="91"/>
+<wire x1="160.02" y1="170.18" x2="195.58" y2="170.18" width="0.1524" layer="91"/>
+<junction x="195.58" y="170.18"/>
 </segment>
 </net>
@@
 <wire x1="83.82" y1="167.64" x2="88.9" y2="167.64" width="0.1524" layer="91" grouprefs="SP32"/>
 <pinref part="ESP32" gate="G$1" pin="EN"/>
-<pinref part="S2" gate="G$1" pin="COM"/>
+<pinref part="RESET" gate="G$1" pin="COM"/>
 <wire x1="88.9" y1="149.86" x2="88.9" y2="167.64" width="0.1524" layer="91"/>
 <label x="109.22" y="167.64" size="1.778" layer="95"/>
@@
 <pinref part="P+2" gate="1" pin="+5V"/>
 <wire x1="297.18" y1="215.9" x2="297.18" y2="213.36" width="0.1524" layer="91"/>
-<pinref part="R3" gate="G$1" pin="2"/>
-<wire x1="297.18" y1="198.12" x2="297.142203125" y2="198.12" width="0.1524" layer="91"/>
-<wire x1="297.142203125" y1="198.12" x2="297.142203125" y2="195.790640625" width="0.1524" layer="91"/>
-<wire x1="297.18" y1="213.36" x2="297.18" y2="198.12" width="0.1524" layer="91"/>
+<pinref part="LED1" gate="G$1" pin="A"/>
+<wire x1="297.18" y1="212.09" x2="297.18" y2="213.36" width="0.1524" layer="91"/>
 </segment>
 <segment>
@@
 <pinref part="VSS5" gate="G$1" pin="VSS"/>
 <wire x1="467.36" y1="195.58" x2="467.36" y2="200.66" width="0.1524" layer="91"/>
+</segment>
+<segment>
+<pinref part="VSS6" gate="G$1" pin="VSS"/>
+<pinref part="R13" gate="G$1" pin="2"/>
+<wire x1="469.9" y1="76.2" x2="469.9" y2="78.74" width="0.1524" layer="91"/>
 </segment>
 </net>
@@
 </segment>
 </net>
+<net name="N$2" class="0">
+<segment>
+<pinref part="LED1" gate="G$1" pin="K"/>
+<pinref part="R3" gate="G$1" pin="2"/>
+<wire x1="297.18" y1="196.85" x2="297.18" y2="195.790640625" width="0.1524" layer="91"/>
+<wire x1="297.18" y1="195.790640625" x2="297.142203125" y2="195.790640625" width="0.1524" layer="91"/>
+</segment>
+</net>
+<net name="N$3" class="0">
+<segment>
+<pinref part="ESP32" gate="G$1" pin="IO48"/>
+<pinref part="LED3" gate="G$1" pin="A"/>
+<wire x1="127" y1="111.76" x2="121.92" y2="111.76" width="0.1524" layer="91"/>
+</segment>
+</net>
+<net name="N$4" class="0">
+<segment>
+<pinref part="ESP32" gate="G$1" pin="IO47"/>
+<pinref part="LED2" gate="G$1" pin="A"/>
+<wire x1="127" y1="114.3" x2="88.9" y2="114.3" width="0.1524" layer="91"/>
+</segment>
+</net>
