File: Electromiografo.brd (EAGLE design)
At the start: 101.3 x 66 mm, 40 parts, among them IC1 ESP32-S3-WROOM-1-N16R8, IC10 LMV321IDBVRG4, IC2 MCP73831T-2DCI_OT, IC4 LP38692MP-3.3_NOPB, IC5 REF2033AIDDCT, IC6 LMV321IDBVRG4, IC7 LMV321IDBVRG4, IC8 LMV321IDBVRG4, IC9 AD8223ARMZ, J1 1981584-1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

Commit message: Se realozaron ajustes finales a la pcb
Parts:
- renumbered IC1 to ESP32, IC4 to REG, IC9 to INA, J1 to USB, J2 to CBAT, S3 to S3-1
Routing:
- net +3V3: track 251.5 -> 253.5 mm

Commit message: fix: PCB reviewed
Parts:
- moved C9 3.00 mm to (43.8, 37.1)
- moved C1 2.35 mm to (62.7, 29.0), turned to 270 degrees
Routing:
- net +3V3: track 253.5 -> 247.7 mm
- net N$38: track 17.6 -> 14.6 mm
- net GND: track 4.07 -> 2.31 mm, vias 106 -> 107
- net N$36: track 19.9 -> 19.1 mm
Changed lines of the file:
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@@
 <setting verticaltext="up"/>
 </settings>
-<grid distance="1" unitdist="mm" unit="mm" style="lines" multiple="1" display="yes" altdistance="2.5" altunitdist="mil" altunit="mil"/>
+<grid distance="39.3700787" unitdist="mil" unit="mil" style="lines" multiple="1" display="yes" altdistance="2.5" altunitdist="mil" altunit="mil"/>
 <layers>
 <layer number="1" name="Top" color="4" fill="1" visible="yes" active="yes"/>
@@
 </autorouter>
 <elements>
-<element name="C1" library="rcl" library_urn="urn:adsk.eagle:library:334" package="C0603" package3d_urn="urn:adsk.eagle:package:23616/2" value="0.1U" x="62.23" y="26.67" smashed="yes">
-<attribute name="NAME" x="60.65656875" y="28.03815" size="1.27" layer="25"/>
-<attribute name="POPULARITY" value="73" x="107.95" y="-33.02" size="1.778" layer="27" display="off"/>
-<attribute name="SPICEPREFIX" value="C" x="107.95" y="-33.02" size="1.778" layer="27" display="off"/>
+<element name="C1" library="rcl" library_urn="urn:adsk.eagle:library:334" package="C0603" package3d_urn="urn:adsk.eagle:package:23616/2" value="0.1U" x="62.67" y="28.9765" smashed="yes" rot="R270">
+<attribute name="NAME" x="64.03815" y="30.54993125" size="1.27" layer="25" rot="R270"/>
+<attribute name="POPULARITY" value="73" x="2.98" y="-16.7435" size="1.778" layer="27" rot="R270" display="off"/>
+<attribute name="SPICEPREFIX" value="C" x="2.98" y="-16.7435" size="1.778" layer="27" rot="R270" display="off"/>
 </element>
 <element name="C10" library="rcl" library_urn="urn:adsk.eagle:library:334" package="C0805" package3d_urn="urn:adsk.eagle:package:23617/2" value="" x="45.6565" y="22.225" smashed="yes" rot="R90">
@@
 <attribute name="VALUE" x="52.07" y="13.97" size="1.27" layer="27" rot="R90"/>
 </element>
-<element name="C9" library="rcl" library_urn="urn:adsk.eagle:library:334" package="C0805" package3d_urn="urn:adsk.eagle:package:23617/2" value="" x="46.7995" y="37.1475" smashed="yes" rot="R90">
-<attribute name="NAME" x="45.265565625" y="34.93906875" size="1.27" layer="25" rot="R90"/>
-<attribute name="POPULARITY" value="88" x="119.1895" y="77.7875" size="1.778" layer="27" rot="R90" display="off"/>
-<attribute name="SPICEPREFIX" value="C" x="119.1895" y="77.7875" size="1.778" layer="27" rot="R90" display="off"/>
-<attribute name="VALUE" x="49.3395" y="35.8775" size="1.27" layer="27" rot="R90"/>
+<element name="C9" library="rcl" library_urn="urn:adsk.eagle:library:334" package="C0805" package3d_urn="urn:adsk.eagle:package:23617/2" value="" x="43.7995" y="37.1475" smashed="yes" rot="R90">
+<attribute name="NAME" x="42.265565625" y="34.93906875" size="1.27" layer="25" rot="R90"/>
+<attribute name="POPULARITY" value="88" x="116.1895" y="77.7875" size="1.778" layer="27" rot="R90" display="off"/>
+<attribute name="SPICEPREFIX" value="C" x="116.1895" y="77.7875" size="1.778" layer="27" rot="R90" display="off"/>
+<attribute name="VALUE" x="46.3395" y="35.8775" size="1.27" layer="27" rot="R90"/>
 </element>
 <element name="ESP32" library="SamacSys_Parts" package="ESP32S3WROOM1N16R8" value="ESP32-S3-WROOM-1-N16R8" x="72.39" y="52.07" smashed="yes">
@@
 <via x="58.6105" y="58.3565" extent="1-16" drill="0.35"/>
 <via x="96.52" y="27.94" extent="1-16" drill="0.35"/>
-<wire x1="96.5755" y1="20.477" x2="97.633" y2="20.477" width="0.3048" layer="1"/>
-<wire x1="97.633" y1="20.477" x2="97.663" y2="20.447" width="0.3048" layer="1"/>
-<wire x1="97.663" y1="20.447" x2="97.70605" y2="20.447" width="0.3048" layer="1"/>
-<wire x1="97.70605" y1="20.447" x2="97.63075" y2="20.5223" width="0.3048" layer="1"/>
 <wire x1="96.5755" y1="20.477" x2="96.6208" y2="20.5223" width="0.3048" layer="1"/>
-<wire x1="97.63075" y1="20.5223" x2="96.6208" y2="20.5223" width="0.3048" layer="1"/>
-<wire x1="96.5755" y1="20.477" x2="95.22" y2="20.477" width="0.3048" layer="1"/>
-<wire x1="95.22" y1="20.477" x2="95.123" y2="20.574" width="0.3048" layer="1"/>
 <via x="3.556" y="51.1175" extent="1-16" drill="0.35"/>
 <via x="4.7625" y="51.1175" extent="1-16" drill="0.35"/>
@@
 <via x="53.7154375" y="1.5875" extent="1-16" drill="0.35"/>
 <via x="54.9854375" y="1.651" extent="1-16" drill="0.35"/>
+<via x="96.17" y="25.86" extent="1-16" drill="0.35"/>
+<wire x1="96.5755" y1="20.477" x2="96.5755" y2="22.152" width="0.3048" layer="1"/>
+<wire x1="96.5755" y1="22.152" x2="96.8005" y2="22.377" width="0.3048" layer="1"/>
 </signal>
 <signal name="N$1">
@@
 <wire x1="55.88" y1="62.23" x2="45.72" y2="62.23" width="0.4064" layer="1"/>
 <wire x1="45.72" y1="62.23" x2="34.29" y2="62.23" width="0.4064" layer="1"/>
-<wire x1="63.08" y1="26.67" x2="66.069325" y2="26.67" width="0.4064" layer="1"/>
 <wire x1="52.07" y1="51.12" x2="46.67" y2="51.12" width="0.4064" layer="1"/>
 <wire x1="46.67" y1="51.12" x2="45.72" y2="52.07" width="0.4064" layer="1"/>
@@
 <wire x1="53.02" y1="21.27" x2="54.61" y2="22.86" width="0.4064" layer="1"/>
 <wire x1="53.02" y1="24.15" x2="53.02" y2="21.27" width="0.4064" layer="1"/>
-<wire x1="57.15" y1="26.67" x2="60.628434375" y2="30.148434375" width="0.4064" layer="1"/>
-<wire x1="60.628434375" y1="30.148434375" x2="63.133421875" y2="30.148434375" width="0.4064" layer="1"/>
-<wire x1="63.133421875" y1="30.148434375" x2="64.443884375" y2="30.147128125" width="0.4064" layer="1"/>
-<wire x1="64.443884375" y1="30.147128125" x2="64.414559375" y2="30.147128125" width="0.4064" layer="1"/>
-<wire x1="64.414559375" y1="30.147128125" x2="65.954175" y2="28.6075125" width="0.4064" layer="1"/>
-<wire x1="65.954175" y1="28.6075125" x2="65.954175" y2="28.59285" width="0.4064" layer="1"/>
-<wire x1="65.954175" y1="28.59285" x2="66.069325" y2="28.4777" width="0.4064" layer="1"/>
-<wire x1="66.069325" y1="28.4777" x2="66.069325" y2="26.67" width="0.4064" layer="1"/>
+<wire x1="57.15" y1="26.67" x2="58.628434375" y2="28.148434375" width="0.4064" layer="1"/>
 <wire x1="74.9282" y1="21.91" x2="74.9307" y2="21.9075" width="0.4064" layer="1"/>
 <wire x1="74.9282" y1="21.91" x2="74.93" y2="21.9118" width="0.4064" layer="1"/>
@@
 <wire x1="74.93" y1="25.4" x2="73.66" y2="26.67" width="0.4064" layer="1"/>
 <wire x1="73.66" y1="26.67" x2="72.39" y2="26.67" width="0.4064" layer="1"/>
-<wire x1="72.39" y1="26.67" x2="66.069325" y2="26.67" width="0.4064" layer="1"/>
+<wire x1="66.069325" y1="26.67" x2="72.39" y2="26.67" width="0.4064" layer="1"/>
 <wire x1="72.39" y1="29.53" x2="72.39" y2="26.67" width="0.4064" layer="1"/>
 <wire x1="35.88" y1="33" x2="33.04" y2="33" width="0.4064" layer="1"/>
@@
 <wire x1="33.02" y1="38.1025" x2="35.5165" y2="38.1025" width="0.4064" layer="1"/>
 <wire x1="33.02" y1="38.1025" x2="33.02" y2="60.96" width="0.4064" layer="1"/>
+<wire x1="62.648065625" y1="28.148434375" x2="62.67" y2="28.1265" width="0.4064" layer="1"/>
+<wire x1="58.628434375" y1="28.148434375" x2="62.648065625" y2="28.148434375" width="0.4064" layer="1"/>
+<wire x1="62.67" y1="28.1265" x2="64.612825" y2="28.1265" width="0.4064" layer="1"/>
+<wire x1="64.612825" y1="28.1265" x2="66.069325" y2="26.67" width="0.4064" layer="1"/>
 </signal>
 <signal name="RESET">
@@
 <contactref element="C8" pad="2"/>
 <contactref element="R9" pad="1"/>
-<wire x1="49.53" y1="16.19" x2="49.53" y2="22.86" width="0.3048" layer="1"/>
-<wire x1="50.82" y1="24.15" x2="51.12" y2="24.15" width="0.3048" layer="1"/>
-<wire x1="49.53" y1="22.86" x2="50.82" y2="24.15" width="0.3048" layer="1"/>
-<wire x1="51.12" y1="26.65" x2="50.78" y2="26.65" width="0.3048" layer="1"/>
-<wire x1="50.78" y1="26.65" x2="49.53" y2="25.4" width="0.3048" layer="1"/>
-<wire x1="49.53" y1="22.86" x2="49.53" y2="25.4" width="0.3048" layer="1"/>
-<wire x1="49.53" y1="25.4" x2="49.53" y2="31.43" width="0.3048" layer="1"/>
+<wire x1="49.53" y1="16.19" x2="49.53" y2="23.86" width="0.3048" layer="1"/>
+<wire x1="49.82" y1="24.15" x2="51.12" y2="24.15" width="0.3048" layer="1"/>
+<wire x1="49.53" y1="23.86" x2="49.82" y2="24.15" width="0.3048" layer="1"/>
+<wire x1="51.12" y1="26.65" x2="49.78" y2="26.65" width="0.3048" layer="1"/>
+<wire x1="49.78" y1="26.65" x2="49.53" y2="26.4" width="0.3048" layer="1"/>
+<wire x1="49.53" y1="23.86" x2="49.53" y2="26.4" width="0.3048" layer="1"/>
+<wire x1="49.53" y1="26.4" x2="49.53" y2="31.43" width="0.3048" layer="1"/>
 <wire x1="49.53" y1="31.43" x2="49.21" y2="31.75" width="0.3048" layer="1"/>
 </signal>
@@
 <contactref element="R10" pad="2"/>
 <wire x1="40.64" y1="25.08" x2="40.64" y2="27.94" width="0.3048" layer="1"/>
-<wire x1="40.64" y1="27.94" x2="44.45" y2="31.75" width="0.3048" layer="1"/>
-<wire x1="44.45" y1="31.75" x2="47.31" y2="31.75" width="0.3048" layer="1"/>
-<wire x1="44.45" y1="31.75" x2="46.7995" y2="34.0995" width="0.3048" layer="1"/>
-<wire x1="46.7995" y1="34.0995" x2="46.7995" y2="36.1975" width="0.3048" layer="1"/>
+<wire x1="40.64" y1="27.94" x2="43.7995" y2="31.0995" width="0.3048" layer="1"/>
+<wire x1="43.7995" y1="31.0995" x2="43.7995" y2="32" width="0.3048" layer="1"/>
+<wire x1="43.7995" y1="32" x2="43.7995" y2="36.1975" width="0.3048" layer="1"/>
+<wire x1="47.31" y1="31.75" x2="47.06" y2="32" width="0.3048" layer="1"/>
+<wire x1="47.06" y1="32" x2="43.7995" y2="32" width="0.3048" layer="1"/>
 </signal>
 <signal name="N$37">
@@
 <wire x1="37.78" y1="30.5" x2="37.78" y2="33" width="0.3048" layer="1"/>
 <wire x1="37.78" y1="35.24" x2="37.78" y2="33" width="0.3048" layer="1"/>
-<wire x1="46.797" y1="38.1" x2="40.64" y2="38.1" width="0.3048" layer="1"/>
-<wire x1="46.797" y1="38.1" x2="46.7995" y2="38.0975" width="0.3048" layer="1"/>
+<wire x1="43.797" y1="38.1" x2="40.64" y2="38.1" width="0.3048" layer="1"/>
+<wire x1="43.797" y1="38.1" x2="43.7995" y2="38.0975" width="0.3048" layer="1"/>
 <wire x1="37.78" y1="35.24" x2="40.64" y2="38.1" width="0.3048" layer="1"/>
 <wire x1="40.64" y1="38.1" x2="40.6425" y2="38.1025" width="0.3048" layer="1"/>

Commit message: Finalizacion de PCB
Parts:
- added LED1, LED2, LED3: HSMW-C170-U0000, SamacSys_Parts:LEDC2012X90N
- moved R13 1.44 mm to (43.0, 43.5), turned to 0 degrees
- moved USB 1.27 mm to (98.0, 19.1)
- renumbered S1 to FLASH, S2 to RESET
Connections:
- new net N$2: LED1.1, R3.2
- new net N$3: ESP32.25, LED3.2
- new net N$4: ESP32.24, LED2.2
- net +5V: now also LED1.2; no longer R3.2
- net GND: now also LED2.1, LED3.1; no longer R13.2
- net N$1: now also ESP32.27; no longer ESP32.26
- net VSS: now also R13.2
Routing:
- net VSS: track 137.7 -> 164.9 mm, vias 2 -> 4
- net N$4: track 0.00 -> 17.6 mm, vias 0 -> 2
- net +5V: track 62.9 -> 45.4 mm
- net N$2: track 0.00 -> 14.7 mm
- net N$3: track 0.00 -> 12.4 mm, vias 0 -> 2
- net N$1: track 69.7 -> 71.7 mm
- net D+: track 43.0 -> 42.2 mm
- net D-: track 44.2 -> 43.5 mm
- net GND: vias 107 -> 103
Other:
- board size 101.3 x 66 mm -> 100 x 66 mm
